File: Ethernet.sch (KiCad schematic (older format))
At the start: 31 parts, among them J1 Wuerth_7499010121A, U3 DP83848C, Y3 25MHz

Commit message: Update footprints
Parts:
- C57, C58, C59, C60, C61, C62, C63, C64, C65, C66, C67: footprint (none) -> Capacitor_SMD:C_0603_1608Metric
- FB2: footprint (none) -> Inductor_SMD:L_0603_1608Metric
- R16, R17: footprint (none) -> Resistor_SMD:R_0603_1608Metric
- R36, R6, R7: footprint (none) -> Resistor_SMD:R_0603_1608Metric_Pad1.05x0.95mm_HandSolder
- R8: footprint Resistor_SMD:R_0603_1608Metric -> Resistor_SMD:R_0603_1608Metric_Pad1.05x0.95mm_HandSolder
- Y3: footprint Crystal:Crystal_SMD_2520-4Pin_2.5x2.0mm -> Crystal:Crystal_SMD_3225-4Pin_3.2x2.5mm
Changed lines of the file:
@@
 F 0 "Y3" H 4650 4850 50  0000 L CNN
 F 1 "25MHz" H 4500 4750 50  0000 L CNN
-F 2 "Crystal:Crystal_SMD_2520-4Pin_2.5x2.0mm" H 4900 4600 50  0001 C CNN
+F 2 "Crystal:Crystal_SMD_3225-4Pin_3.2x2.5mm" H 4900 4600 50  0001 C CNN
 F 3 "~" H 4900 4600 50  0001 C CNN
 	1    4900 4600
@@
 F 0 "R8" V 5450 4700 50  0000 C CNN
 F 1 "0" V 5450 4600 50  0000 C CNN
-F 2 "Resistor_SMD:R_0603_1608Metric" V 5480 4600 50  0001 C CNN
+F 2 "Resistor_SMD:R_0603_1608Metric_Pad1.05x0.95mm_HandSolder" V 5480 4600 50  0001 C CNN
 F 3 "~" H 5550 4600 50  0001 C CNN
 	1    5550 4600
@@
 F 0 "C62" H 4515 6046 50  0000 L CNN
 F 1 "10u" H 4515 5955 50  0000 L CNN
-F 2 "" H 4438 5850 50  0001 C CNN
+F 2 "Capacitor_SMD:C_0603_1608Metric" H 4438 5850 50  0001 C CNN
 F 3 "~" H 4400 6000 50  0001 C CNN
 	1    4400 6000
@@
 F 0 "C63" H 4865 6046 50  0000 L CNN
 F 1 "100n" H 4865 5955 50  0000 L CNN
-F 2 "" H 4788 5850 50  0001 C CNN
+F 2 "Capacitor_SMD:C_0603_1608Metric" H 4788 5850 50  0001 C CNN
 F 3 "~" H 4750 6000 50  0001 C CNN
 	1    4750 6000
@@
 F 0 "C64" H 5315 6046 50  0000 L CNN
 F 1 "100n" H 5315 5955 50  0000 L CNN
-F 2 "" H 5238 5850 50  0001 C CNN
+F 2 "Capacitor_SMD:C_0603_1608Metric" H 5238 5850 50  0001 C CNN
 F 3 "~" H 5200 6000 50  0001 C CNN
 	1    5200 6000
@@
 F 0 "C65" H 5715 6046 50  0000 L CNN
 F 1 "100n" H 5715 5955 50  0000 L CNN
-F 2 "" H 5638 5850 50  0001 C CNN
+F 2 "Capacitor_SMD:C_0603_1608Metric" H 5638 5850 50  0001 C CNN
 F 3 "~" H 5600 6000 50  0001 C CNN
 	1    5600 6000
@@
 F 0 "FB2" V 8826 5650 50  0000 C CNN
 F 1 "Ferrite_Bead" V 8917 5650 50  0000 C CNN
-F 2 "" V 9030 5650 50  0001 C CNN
+F 2 "Inductor_SMD:L_0603_1608Metric" V 9030 5650 50  0001 C CNN
 F 3 "~" H 9100 5650 50  0001 C CNN
 	1    9100 5650
@@
 F 0 "C66" H 9365 5846 50  0000 L CNN
 F 1 "100n" H 9365 5755 50  0000 L CNN
-F 2 "" H 9288 5650 50  0001 C CNN
+F 2 "Capacitor_SMD:C_0603_1608Metric" H 9288 5650 50  0001 C CNN
 F 3 "~" H 9250 5800 50  0001 C CNN
 	1    9250 5800
@@
 F 0 "C67" H 9765 5846 50  0000 L CNN
 F 1 "10n" H 9765 5755 50  0000 L CNN
-F 2 "" H 9688 5650 50  0001 C CNN
+F 2 "Capacitor_SMD:C_0603_1608Metric" H 9688 5650 50  0001 C CNN
 F 3 "~" H 9650 5800 50  0001 C CNN
 	1    9650 5800
@@
 F 0 "C57" H 1615 5596 50  0000 L CNN
 F 1 "10u" H 1615 5505 50  0000 L CNN
-F 2 "" H 1538 5400 50  0001 C CNN
+F 2 "Capacitor_SMD:C_0603_1608Metric" H 1538 5400 50  0001 C CNN
 F 3 "~" H 1500 5550 50  0001 C CNN
 	1    1500 5550
@@
 F 0 "C58" H 1965 5596 50  0000 L CNN
 F 1 "100n" H 1965 5505 50  0000 L CNN
-F 2 "" H 1888 5400 50  0001 C CNN
+F 2 "Capacitor_SMD:C_0603_1608Metric" H 1888 5400 50  0001 C CNN
 F 3 "~" H 1850 5550 50  0001 C CNN
 	1    1850 5550
@@
 F 0 "C59" H 2315 5596 50  0000 L CNN
 F 1 "100n" H 2315 5505 50  0000 L CNN
-F 2 "" H 2238 5400 50  0001 C CNN
+F 2 "Capacitor_SMD:C_0603_1608Metric" H 2238 5400 50  0001 C CNN
 F 3 "~" H 2200 5550 50  0001 C CNN
 	1    2200 5550
@@
 F 0 "C60" H 2865 5596 50  0000 L CNN
 F 1 "100n" H 2865 5505 50  0000 L CNN
-F 2 "" H 2788 5400 50  0001 C CNN
+F 2 "Capacitor_SMD:C_0603_1608Metric" H 2788 5400 50  0001 C CNN
 F 3 "~" H 2750 5550 50  0001 C CNN
 	1    2750 5550
@@
 F 0 "C61" H 3315 5596 50  0000 L CNN
 F 1 "10u" H 3315 5505 50  0000 L CNN
-F 2 "" H 3238 5400 50  0001 C CNN
+F 2 "Capacitor_SMD:C_0603_1608Metric" H 3238 5400 50  0001 C CNN
 F 3 "~" H 3200 5550 50  0001 C CNN
 	1    3200 5550
@@
 F 0 "R7" H 2170 4446 50  0000 L CNN
 F 1 "470" H 2170 4355 50  0000 L CNN
-F 2 "" V 2030 4400 50  0001 C CNN
+F 2 "Resistor_SMD:R_0603_1608Metric_Pad1.05x0.95mm_HandSolder" V 2030 4400 50  0001 C CNN
 F 3 "~" H 2100 4400 50  0001 C CNN
 	1    2100 4400
@@
 F 0 "R16" H 2920 4046 50  0000 L CNN
 F 1 "220" H 2920 3955 50  0000 L CNN
-F 2 "" V 2780 4000 50  0001 C CNN
+F 2 "Resistor_SMD:R_0603_1608Metric" V 2780 4000 50  0001 C CNN
 F 3 "~" H 2850 4000 50  0001 C CNN
 	1    2850 4000
@@
 F 0 "R17" H 2920 4446 50  0000 L CNN
 F 1 "470" H 2920 4355 50  0000 L CNN
-F 2 "" V 2780 4400 50  0001 C CNN
+F 2 "Resistor_SMD:R_0603_1608Metric" V 2780 4400 50  0001 C CNN
 F 3 "~" H 2850 4400 50  0001 C CNN
 	1    2850 4400
@@
 F 0 "R6" H 2170 4046 50  0000 L CNN
 F 1 "220" H 2170 3955 50  0000 L CNN
-F 2 "" V 2030 4000 50  0001 C CNN
+F 2 "Resistor_SMD:R_0603_1608Metric_Pad1.05x0.95mm_HandSolder" V 2030 4000 50  0001 C CNN
 F 3 "~" H 2100 4000 50  0001 C CNN
 	1    2100 4000
@@
 F 0 "R36" H 6870 4096 50  0000 L CNN
 F 1 "DNP" H 6870 4005 50  0000 L CNN
-F 2 "" V 6730 4050 50  0001 C CNN
+F 2 "Resistor_SMD:R_0603_1608Metric_Pad1.05x0.95mm_HandSolder" V 6730 4050 50  0001 C CNN
 F 3 "~" H 6800 4050 50  0001 C CNN
 	1    6800 4050
