File: RAM.sch (KiCad schematic (older format))
At the start: 20 parts, among them J5 Conn_ARM_JTAG_SWD_20, SW4 SW_Push, U1 STM32MP151AAB3, U2 MT41K64M16TW-107_AAT_J_TR

Commit message: Complete schematic rough draft
Connections:
- net 3V3: now also U1.T15 (BYPASS_REG1V8)
- net GND: no longer U1.T15 (BYPASS_REG1V8)
- net A13: no longer names the net of U1.F17 (DDR_A13)
- net A14: no longer names the net of U1.N18 (DDR_A14)
- net A15: no longer names the net of U1.L16 (DDR_A15)
- no-connect marks 5 -> 8
Changed lines of the file:
@@
 Text Label 4200 2000 0    50   ~ 0
 A11
-Text Label 4850 2600 2    50   ~ 0
-A15
-Text Label 4850 2500 2    50   ~ 0
-A14
-Text Label 4850 2400 2    50   ~ 0
-A13
 Text Label 4850 2300 2    50   ~ 0
 A12
@@
 Text Label 7250 2800 0    50   ~ 0
 LDM
-Text Label 8050 2750 2    50   ~ 0
-DDRVREF
 Text Label 8050 2950 2    50   ~ 0
 CK_N
@@
 	1    0    0    -1
 $EndComp
-Text Label 10750 1750 0    50   ~ 0
-3V3
 Text Label 10750 3350 0    50   ~ 0
 3V3
@@
 $EndComp
 Connection ~ 10550 4500
-Text Label 10550 4200 0    50   ~ 0
-3V3
 $Comp
 L Connector:Conn_ARM_JTAG_SWD_20 J5
@@
 	1    0    0    -1
 $EndComp
-Text Label 8000 4200 0    50   ~ 0
-3V3
 Wire Wire Line
 	8000 4200 8000 4350
@@
 Reset Button\n
 $Comp
-L power:GND #PWR035
-U 1 1 614383F1
-P 8050 3450
-F 0 "#PWR035" H 8050 3200 50  0001 C CNN
-F 1 "GND" H 8055 3277 50  0000 C CNN
-F 2 "" H 8050 3450 50  0001 C CNN
-F 3 "" H 8050 3450 50  0001 C CNN
-	1    8050 3450
-	1    0    0    -1
-$EndComp
-$Comp
 L Device:R R33
 U 1 1 61444559
@@
 Text Notes 3450 7100 0    50   ~ 0
 NOTE not 3v3\n
+Text Label 8050 2750 2    50   ~ 0
+DDRVREF
+Text HLabel 8000 4200 0    50   Input ~ 0
+3V3
+Text HLabel 10550 4200 0    50   Input ~ 0
+3V3
+Text HLabel 10750 1750 2    50   Input ~ 0
+3V3
+Text HLabel 8050 3450 0    50   Input ~ 0
+3V3
+NoConn ~ 4850 2500
+NoConn ~ 4850 2600
+NoConn ~ 4850 2400
 $EndSCHEMATC

Commit message: Update footprints
Parts:
- C85, C86, C87, C88, C89, C90, C91, C92: footprint (none) -> Capacitor_SMD:C_0603_1608Metric
- J5: footprint (none) -> Connector_PinHeader_1.27mm:PinHeader_2x10_P1.27mm_Vertical
- R18, R29, R30, R31, R32: footprint (none) -> Resistor_SMD:R_0603_1608Metric_Pad1.05x0.95mm_HandSolder
- R19, R20, R33: footprint (none) -> Resistor_SMD:R_0603_1608Metric
- SW4: footprint (none) -> Button_Switch_SMD:SW_Push_1P1T_NO_6x6mm_H9.5mm
Changed lines of the file:
@@
 F 0 "R18" H 5320 4396 50  0000 L CNN
 F 1 "10k" H 5320 4305 50  0000 L CNN
-F 2 "" V 5180 4350 50  0001 C CNN
+F 2 "Resistor_SMD:R_0603_1608Metric_Pad1.05x0.95mm_HandSolder" V 5180 4350 50  0001 C CNN
 F 3 "~" H 5250 4350 50  0001 C CNN
 	1    5250 4350
@@
 F 0 "C85" H 5115 7096 50  0000 L CNN
 F 1 "100n" H 5115 7005 50  0000 L CNN
-F 2 "" H 5038 6900 50  0001 C CNN
+F 2 "Capacitor_SMD:C_0603_1608Metric" H 5038 6900 50  0001 C CNN
 F 3 "~" H 5000 7050 50  0001 C CNN
 	1    5000 7050
@@
 F 0 "C86" H 5465 7096 50  0000 L CNN
 F 1 "100n" H 5465 7005 50  0000 L CNN
-F 2 "" H 5388 6900 50  0001 C CNN
+F 2 "Capacitor_SMD:C_0603_1608Metric" H 5388 6900 50  0001 C CNN
 F 3 "~" H 5350 7050 50  0001 C CNN
 	1    5350 7050
@@
 F 0 "C87" H 5815 7096 50  0000 L CNN
 F 1 "100n" H 5815 7005 50  0000 L CNN
-F 2 "" H 5738 6900 50  0001 C CNN
+F 2 "Capacitor_SMD:C_0603_1608Metric" H 5738 6900 50  0001 C CNN
 F 3 "~" H 5700 7050 50  0001 C CNN
 	1    5700 7050
@@
 F 0 "R19" H 5770 4396 50  0000 L CNN
 F 1 "240" H 5770 4305 50  0000 L CNN
-F 2 "" V 5630 4350 50  0001 C CNN
+F 2 "Resistor_SMD:R_0603_1608Metric" V 5630 4350 50  0001 C CNN
 F 3 "~" H 5700 4350 50  0001 C CNN
 	1    5700 4350
@@
 F 0 "R20" H 6220 4396 50  0000 L CNN
 F 1 "240" H 6220 4305 50  0000 L CNN
-F 2 "" V 6080 4350 50  0001 C CNN
+F 2 "Resistor_SMD:R_0603_1608Metric" V 6080 4350 50  0001 C CNN
 F 3 "~" H 6150 4350 50  0001 C CNN
 	1    6150 4350
@@
 F 0 "C88" H 1165 7096 50  0000 L CNN
 F 1 "100n" H 1165 7005 50  0000 L CNN
-F 2 "" H 1088 6900 50  0001 C CNN
+F 2 "Capacitor_SMD:C_0603_1608Metric" H 1088 6900 50  0001 C CNN
 F 3 "~" H 1050 7050 50  0001 C CNN
 	1    1050 7050
@@
 F 0 "C89" H 1615 7096 50  0000 L CNN
 F 1 "100n" H 1615 7005 50  0000 L CNN
-F 2 "" H 1538 6900 50  0001 C CNN
+F 2 "Capacitor_SMD:C_0603_1608Metric" H 1538 6900 50  0001 C CNN
 F 3 "~" H 1500 7050 50  0001 C CNN
 	1    1500 7050
@@
 F 0 "C90" H 2015 7096 50  0000 L CNN
 F 1 "100n" H 2015 7005 50  0000 L CNN
-F 2 "" H 1938 6900 50  0001 C CNN
+F 2 "Capacitor_SMD:C_0603_1608Metric" H 1938 6900 50  0001 C CNN
 F 3 "~" H 1900 7050 50  0001 C CNN
 	1    1900 7050
@@
 F 0 "C91" H 2415 7096 50  0000 L CNN
 F 1 "100n" H 2415 7005 50  0000 L CNN
-F 2 "" H 2338 6900 50  0001 C CNN
+F 2 "Capacitor_SMD:C_0603_1608Metric" H 2338 6900 50  0001 C CNN
 F 3 "~" H 2300 7050 50  0001 C CNN
 	1    2300 7050
@@
 F 0 "C92" H 10315 4696 50  0000 L CNN
 F 1 "C" H 10315 4605 50  0000 L CNN
-F 2 "" H 10238 4500 50  0001 C CNN
+F 2 "Capacitor_SMD:C_0603_1608Metric" H 10238 4500 50  0001 C CNN
 F 3 "~" H 10200 4650 50  0001 C CNN
 	1    10200 4650
@@
 F 0 "SW4" V 10504 4848 50  0000 L CNN
 F 1 "SW_Push" V 10595 4848 50  0000 L CNN
-F 2 "" H 10550 4900 50  0001 C CNN
+F 2 "Button_Switch_SMD:SW_Push_1P1T_NO_6x6mm_H9.5mm" H 10550 4900 50  0001 C CNN
 F 3 "~" H 10550 4900 50  0001 C CNN
 	1    10550 4700
@@
 F 0 "R32" H 10620 4396 50  0000 L CNN
 F 1 "10k" H 10620 4305 50  0000 L CNN
-F 2 "" V 10480 4350 50  0001 C CNN
+F 2 "Resistor_SMD:R_0603_1608Metric_Pad1.05x0.95mm_HandSolder" V 10480 4350 50  0001 C CNN
 F 3 "~" H 10550 4350 50  0001 C CNN
 	1    10550 4350
@@
 F 0 "J5" H 7571 5196 50  0000 R CNN
 F 1 "Conn_ARM_JTAG_SWD_20" H 9150 5950 50  0000 R CNN
-F 2 "" H 8550 4100 50  0001 L TNN
+F 2 "Connector_PinHeader_1.27mm:PinHeader_2x10_P1.27mm_Vertical" H 8550 4100 50  0001 L TNN
 F 3 "http://infocenter.arm.com/help/topic/com.arm.doc.dui0499b/DUI0499B_system_design_reference.pdf" V 7750 3900 50  0001 C CNN
 	1    8100 5150
@@
 F 0 "R30" H 9120 5846 50  0000 L CNN
 F 1 "10K" H 9120 5755 50  0000 L CNN
-F 2 "" V 8980 5800 50  0001 C CNN
+F 2 "Resistor_SMD:R_0603_1608Metric_Pad1.05x0.95mm_HandSolder" V 8980 5800 50  0001 C CNN
 F 3 "~" H 9050 5800 50  0001 C CNN
 	1    9050 5800
@@
 F 0 "R29" H 8870 5846 50  0000 L CNN
 F 1 "10k" H 8870 5755 50  0000 L CNN
-F 2 "" V 8730 5800 50  0001 C CNN
+F 2 "Resistor_SMD:R_0603_1608Metric_Pad1.05x0.95mm_HandSolder" V 8730 5800 50  0001 C CNN
 F 3 "~" H 8800 5800 50  0001 C CNN
 	1    8800 5800
@@
 F 0 "R31" H 9370 5846 50  0000 L CNN
 F 1 "10K" H 9370 5755 50  0000 L CNN
-F 2 "" V 9230 5800 50  0001 C CNN
+F 2 "Resistor_SMD:R_0603_1608Metric_Pad1.05x0.95mm_HandSolder" V 9230 5800 50  0001 C CNN
 F 3 "~" H 9300 5800 50  0001 C CNN
 	1    9300 5800
@@
 F 0 "R33" H 6620 4396 50  0000 L CNN
 F 1 "3K" H 6620 4305 50  0000 L CNN
-F 2 "" V 6480 4350 50  0001 C CNN
+F 2 "Resistor_SMD:R_0603_1608Metric" V 6480 4350 50  0001 C CNN
 F 3 "~" H 6550 4350 50  0001 C CNN
 	1    6550 4350
