File: LinuxBoard/LinuxBoard.kicad_pcb (KiCad board)
At the start: 4 copper layers, 183 parts, among them J1 Wuerth_7499010121A, J2 Conn_02x10_Counter_Clockwise, J3 Micro_SD_Card, J4 USB_A, J5 Conn_ARM_JTAG_SWD_10, J6 USB_B_Micro, J7 Barrel_Jack_Switch, SW1 SW_DIP_x03, SW2 SW_Push, SW3 SW_Push, SW4 SW_Push, SW5 SW_Push, U1 STM32MP151AAB3, U2 MT41K64M16TW-107_AAT_J_TR, U3 DP83848C, U4 STPMIC1APQR, Y1 24MHz, Y2 32.768KHz, Y3 25MHz

Commit message: Fix resistor footprints, restart layout
Parts:
- removed FB4: Ferrite_Bead, Inductor_SMD:L_0603_1608Metric
- added FB3: FerriteBead, Inductor_SMD:L_0603_1608Metric_Pad1.05x0.95mm_HandSolder, F.Cu at (157.9, 67.1)
- added R31: 50k, Resistor_SMD:R_0603_1608Metric_Pad0.98x0.95mm_HandSolder, F.Cu at (77.4, 96.7)
- added R37: 50k, Resistor_SMD:R_0603_1608Metric_Pad0.98x0.95mm_HandSolder, F.Cu at (121.0, 66.7)
- added R38: 50k, Resistor_SMD:R_0603_1608Metric_Pad0.98x0.95mm_HandSolder, F.Cu at (73.1, 94.2)
- added R39: 50k, Resistor_SMD:R_0603_1608Metric_Pad0.98x0.95mm_HandSolder, F.Cu at (73.1, 96.7)
- added R40: 50k, Resistor_SMD:R_0603_1608Metric_Pad0.98x0.95mm_HandSolder, F.Cu at (77.4, 94.2)
- added TP15: TestPoint, TestPoint:TestPoint_Pad_D2.0mm, F.Cu at (148.7, 110.1)
- C16, C17, C18, C19, C20, C21, C22, C23, C24, C25, C26, C27, C28, C29, C30, C31, C32, C33, C34, C35, C36, C37, C38, C39, C40, C41, C42, C43, C44, C45, C46, C47, C48, C49, C50, C51, C52, C53, C54, C55, C56, C85, C86, C87, C88, C89, C90, C91, C93, C94, L6: moved to F.Cu
- FB1, FB2: value Ferrite_Bead -> FerriteBead; footprint Inductor_SMD:L_0603_1608Metric -> Inductor_SMD:L_0603_1608Metric_Pad1.05x0.95mm_HandSolder
- R1, R14, R15, R2, R21, R22, R23, R24, R25, R26, R27, R28, R29, R3, R30, R32, R34, R35, R36, R4, R5, R6, R7, R8: footprint Resistor_SMD:R_0603_1608Metric_Pad1.05x0.95mm_HandSolder -> Resistor_SMD:R_0603_1608Metric_Pad0.98x0.95mm_HandSolder
- R10, R11, R12, R13, R16, R17, R9: footprint Resistor_SMD:R_0603_1608Metric -> Resistor_SMD:R_0603_1608Metric_Pad0.98x0.95mm_HandSolder
- R18: footprint Resistor_SMD:R_0603_1608Metric_Pad1.05x0.95mm_HandSolder -> Resistor_SMD:R_0603_1608Metric_Pad0.98x0.95mm_HandSolder; moved to F.Cu
- R19, R20, R33: footprint Resistor_SMD:R_0603_1608Metric -> Resistor_SMD:R_0603_1608Metric_Pad0.98x0.95mm_HandSolder; moved to F.Cu
- U3: footprint Package_QFP:LQFP-48-1EP_7x7mm_P0.5mm_EP3.6x3.6mm -> Package_QFP:LQFP-48_7x7mm_P0.5mm
- moved F2 154.5 mm to (179.8, 59.1), turned to 0 degrees
- moved J6 144.4 mm to (160.4, 61.7), turned to 0 degrees
- moved R35 143.5 mm to (167.3, 59.1), turned to 0 degrees
- moved R18 142.8 mm to (212.9, 59.1)
- moved D6 140.7 mm to (167.1, 61.7), turned to 0 degrees
- moved F1 138.4 mm to (165.7, 73.3), turned to 0 degrees
- moved R15 137.3 mm to (162.2, 67.1)
- moved J7 136.0 mm to (149.0, 59.8), turned to 0 degrees
- moved R14 135.5 mm to (157.9, 69.6)
- moved TP1 134.7 mm to (167.1, 65.0), turned to 0 degrees
- moved R33 134.6 mm to (208.5, 59.1)
- moved D3 133.7 mm to (157.7, 72.1), turned to 0 degrees
- moved D5 131.2 mm to (175.2, 61.7)
- moved D4 130.5 mm to (171.2, 61.7)
- moved C85 130.3 mm to (208.3, 66.6)
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Connections:
- net /MPU/ETH1_MDC renamed /Ethernet/MDC
- net /MPU/ETH1_MDIO renamed /Ethernet/MDIO
- net /MPU/ETH1_PHY_INTN renamed /Ethernet/ETH_PWR_DOWN
- net /MPU/ETH1_RXD0 renamed /Ethernet/RXD_0
- net /MPU/ETH1_RXD1 renamed /Ethernet/RXD_1
- net /MPU/ETH1_RXD2 renamed /Ethernet/RXD_2
- net /MPU/ETH1_RXD3 renamed /Ethernet/RXD_3
- net /MPU/ETH1_RX_CLK renamed /Ethernet/RX_CLK
- net /MPU/ETH1_RX_DV renamed /Ethernet/RX_DV
- net /MPU/ETH1_RX_ER renamed /Ethernet/RX_ER
- net /MPU/ETH1_TXD0 renamed /Ethernet/TXD_0
- net /MPU/ETH1_TXD1 renamed /Ethernet/TXD_1
- net /MPU/ETH1_TXD2 renamed /Ethernet/TXD_2
- net /MPU/ETH1_TXD3 renamed /Ethernet/TXD_3
- net /MPU/ETH1_TX_CLK renamed /Ethernet/TX_CLK
- net /MPU/ETH1_TX_EN renamed /Ethernet/TX_EN
- net /MPU/ETH_RESETN renamed /Ethernet/ETH_RESET_N
- net /MPU_Power/PMIC_VDD_CORE renamed /MPU_Power/VDD_CORE
- net /MPU_Power/USB_3V3 renamed /PMIC/LDO4OUT
- net /PMIC/VOUT_LDO1 renamed /PMIC/LDO1OUT
- net /PMIC/VOUT_LDO2 renamed /PMIC/LDO2OUT
- net /PMIC/VOUT_LDO5 renamed /PMIC/LDO5OUT
- net /PMIC/VOUT_LDO6 renamed /PMIC/LDO6OUT
- net /PMIC/VTT_DDR3 renamed /PMIC/LDO3OUT
- net /RAM/PMIC_DDR_VREF renamed /PMIC/VREFDDR
- net /RAM/VBUSOTG renamed /PMIC/VBUSOTG
- FB1 pad 1: Net-(F1-Pad2) -> /VDD
- FB1 pad 2: Net-(FB1-Pad2) -> /Ethernet/AVDD33
- FB2 pad 1: /Ethernet/AVDD33 -> Net-(FB2-Pad1)
- FB2 pad 2: /VDD -> Net-(F2-Pad2)
- J5 pad 7: Net-(J5-Pad7) -> unconnected-(J5-Pad7)
- J5 pad 8: Net-(J5-Pad8) -> unconnected-(J5-Pad8)
- J6 pad 1: Net-(FB1-Pad2) -> Net-(FB3-Pad1)
- J6 pad 4: Net-(J6-Pad4) -> unconnected-(J6-Pad4)
- J7 pad 1: Net-(FB4-Pad2) -> Net-(FB2-Pad1)
- R35 pad 2: Net-(FB1-Pad2) -> Net-(FB3-Pad1)
- U1 pad A12: Net-(U1-PadA12) -> unconnected-(U1-PadA12)
- U1 pad A13: Net-(U1-PadA13) -> unconnected-(U1-PadA13)
- U1 pad A14: Net-(U1-PadA14) -> unconnected-(U1-PadA14)
- U1 pad A15: Net-(U1-PadA15) -> unconnected-(U1-PadA15)
- U1 pad A16: Net-(U1-PadA16) -> unconnected-(U1-PadA16)
- U1 pad A3: Net-(U1-PadA3) -> unconnected-(U1-PadA3)
- U1 pad A4: Net-(U1-PadA4) -> unconnected-(U1-PadA4)
- U1 pad A5: Net-(U1-PadA5) -> unconnected-(U1-PadA5)
- U1 pad A6: Net-(U1-PadA6) -> unconnected-(U1-PadA6)
- U1 pad A9: Net-(U1-PadA9) -> unconnected-(U1-PadA9)
- U1 pad B1: Net-(U1-PadB1) -> unconnected-(U1-PadB1)
- U1 pad B11: Net-(U1-PadB11) -> unconnected-(U1-PadB11)
- U1 pad B12: Net-(U1-PadB12) -> unconnected-(U1-PadB12)
- U1 pad B13: Net-(U1-PadB13) -> unconnected-(U1-PadB13)
- U1 pad B14: Net-(U1-PadB14) -> unconnected-(U1-PadB14)
- U1 pad B15: Net-(U1-PadB15) -> unconnected-(U1-PadB15)
- U1 pad B16: Net-(U1-PadB16) -> unconnected-(U1-PadB16)
- U1 pad B7: Net-(U1-PadB7) -> unconnected-(U1-PadB7)
- U1 pad B8: Net-(U1-PadB8) -> unconnected-(U1-PadB8)
- U1 pad C1: Net-(U1-PadC1) -> unconnected-(U1-PadC1)
- U1 pad C2: Net-(U1-PadC2) -> unconnected-(U1-PadC2)
- U1 pad C4: Net-(U1-PadC4) -> unconnected-(U1-PadC4)
- U1 pad C7: Net-(U1-PadC7) -> unconnected-(U1-PadC7)
- U1 pad C9: Net-(U1-PadC9) -> unconnected-(U1-PadC9)
- U1 pad D10: Net-(U1-PadD10) -> unconnected-(U1-PadD10)
- U1 pad D11: Net-(U1-PadD11) -> unconnected-(U1-PadD11)
- U1 pad D12: Net-(U1-PadD12) -> unconnected-(U1-PadD12)
- U1 pad D13: Net-(U1-PadD13) -> unconnected-(U1-PadD13)
- U1 pad D3: Net-(U1-PadD3) -> unconnected-(U1-PadD3)
- U1 pad D9: Net-(U1-PadD9) -> unconnected-(U1-PadD9)
- U1 pad E1: Net-(U1-PadE1) -> unconnected-(U1-PadE1)
- U1 pad F17: Net-(U1-PadF17) -> unconnected-(U1-PadF17)
- U1 pad J19: Net-(U1-PadJ19) -> unconnected-(U1-PadJ19)
- U1 pad K18: Net-(U1-PadK18) -> unconnected-(U1-PadK18)
- U1 pad L16: Net-(U1-PadL16) -> unconnected-(U1-PadL16)
- U1 pad N18: Net-(U1-PadN18) -> unconnected-(U1-PadN18)
- U1 pad N19: Net-(U1-PadN19) -> unconnected-(U1-PadN19)
- U1 pad P1: Net-(U1-PadP1) -> unconnected-(U1-PadP1)
- U1 pad P2: Net-(U1-PadP2) -> unconnected-(U1-PadP2)
- U1 pad R1: Net-(U1-PadR1) -> unconnected-(U1-PadR1)
- U1 pad T10: Net-(U1-PadT10) -> unconnected-(U1-PadT10)
- U1 pad T11: Net-(U1-PadT11) -> unconnected-(U1-PadT11)
- U1 pad T13: Net-(U1-PadT13) -> unconnected-(U1-PadT13)
- U1 pad T14: Net-(U1-PadT14) -> unconnected-(U1-PadT14)
- U1 pad T16: Net-(U1-PadT16) -> unconnected-(U1-PadT16)
- U1 pad T5: Net-(U1-PadT5) -> unconnected-(U1-PadT5)
- U1 pad T7: Net-(U1-PadT7) -> unconnected-(U1-PadT7)
- U1 pad U1: Net-(U1-PadU1) -> unconnected-(U1-PadU1)
- U1 pad U10: Net-(U1-PadU10) -> unconnected-(U1-PadU10)
- U1 pad U16: Net-(U1-PadU16) -> unconnected-(U1-PadU16)
- U1 pad U7: Net-(U1-PadU7) -> unconnected-(U1-PadU7)
- U1 pad U9: Net-(U1-PadU9) -> unconnected-(U1-PadU9)
- U1 pad V10: Net-(U1-PadV10) -> unconnected-(U1-PadV10)
- U1 pad V17: Net-(U1-PadV17) -> unconnected-(U1-PadV17)
- U1 pad V5: Net-(U1-PadV5) -> unconnected-(U1-PadV5)
- U1 pad V7: Net-(U1-PadV7) -> unconnected-(U1-PadV7)
- U1 pad W10: Net-(U1-PadW10) -> unconnected-(U1-PadW10)
- U1 pad W6: Net-(U1-PadW6) -> unconnected-(U1-PadW6)
- U1 pad W7: Net-(U1-PadW7) -> unconnected-(U1-PadW7)
- U1 pad W9: Net-(U1-PadW9) -> unconnected-(U1-PadW9)
- U2 pad J1: Net-(U2-PadJ1) -> unconnected-(U2-PadJ1)
- U2 pad J9: Net-(U2-PadJ9) -> unconnected-(U2-PadJ9)
- U2 pad L1: Net-(U2-PadL1) -> unconnected-(U2-PadL1)
- U2 pad L9: Net-(U2-PadL9) -> unconnected-(U2-PadL9)
- U2 pad M7: Net-(U2-PadM7) -> unconnected-(U2-PadM7)
- U2 pad T3: Net-(U2-PadT3) -> unconnected-(U2-PadT3)
- U2 pad T7: Net-(U2-PadT7) -> unconnected-(U2-PadT7)
- U3 pad 27: Net-(U3-Pad27) -> unconnected-(U3-Pad27)
Routing:
- net GND: track 86.0 -> 0.00 mm, vias 109 -> 0
- net /MPU_Power/VDD_CORE: track 18.9 -> 0.00 mm, vias 34 -> 0
- net /MPU_Power/VDDQ_DDR: track 15.5 -> 0.00 mm, vias 29 -> 0
- net /VDD: track 14.3 -> 0.00 mm, vias 19 -> 0
- net /RAM/NRST: track 4.28 -> 0.00 mm
- net /RAM/A2: track 2.91 -> 0.00 mm, vias 1 -> 0
- net /RAM/DQ8: track 2.90 -> 0.00 mm, vias 1 -> 0
- net /RAM/A0: track 2.87 -> 0.00 mm, vias 1 -> 0
- net /RAM/DQ13: track 2.87 -> 0.00 mm, vias 1 -> 0
- net /RAM/A11: track 2.85 -> 0.00 mm, vias 1 -> 0
- net /RAM/DQ7: track 2.85 -> 0.00 mm, vias 1 -> 0
- net /RAM/CS_N: track 2.84 -> 0.00 mm, vias 1 -> 0
- net /RAM/DQ14: track 2.82 -> 0.00 mm, vias 1 -> 0
- net /RAM/RAS_N: track 2.81 -> 0.00 mm, vias 1 -> 0
- net /RAM/LDM: track 2.81 -> 0.00 mm, vias 1 -> 0
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Other:
- copper layers 4 -> 2
- net class Default removed
- net class JLC removed
- rule pad_to_mask_clearance: 0.051 -> 0
